File: Board/test-end-a/test-end-a.kicad_pcb (KiCad board)
At the start: 2 copper layers, 105 x 80 mm, 49 parts, among them J10 SW2, J11 TENDA_2, J12 TENDA_1, J2 I2C connector, J5 VAC 230V, J7 SW1, J8 Anemometer, J9 TX RX - + Serial TTL, K1 FINDER-36.11, K2 FINDER-36.11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

Commit message: [FIX] Stable version
Parts:
- J9: value TX RX - + Serial TTL -> TX RX - +
- moved C6 2.37 mm to (100.1, 121.1)
- moved C5 2.29 mm to (74.9, 121.4)
- moved C7 1.78 mm to (86.9, 121.9)
Routing:
- net +5V: track 196.4 -> 193.6 mm
- net Net-(J10-Pin_1): track 85.8 -> 87.2 mm
- net GND: track 384.8 -> 385.7 mm
Other:
- board text added: "C"
- board text added: "F1"
- board text added: "F2"
- board text added: "L"
- board text added: "N"
